File: Hardware/Schematic.sch (EAGLE design)
At the start: 103 parts, among them IC1 BD5229G-TR, IC4 XC6220A331MR-G, J1 FH34SRJ-24S-0.5SH_99_, J2 SAMACSYS_PARTS_USB4110-GF-A, J3 QWIIC_RIGHT_ANGLE, J4 112A-TAAR-R03_ATTEND, Q1 20V/4.2A/52mΩ/1.4W, Q2 20V/4.2A/52mΩ/1.4W, Q3 SI1308EDL-T1-GE3, U1 W25Q512JVEIQ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

Commit message: Schematic fixes.
Fixed some junctions not being properly connected.
Added missing component values.

Signed-off-by: Andrei Stan <standrei2003@yahoo.com>
Parts:
- removed C10_SUPERCAP: CPH3225A, DeskAssistant v19 v1:CPH3225A
- R3: value (none) -> 0.47
- SJ1: value (none) -> 0
Connections:
- net GND: no longer C10_SUPERCAP.1
- net VRTC: no longer C10_SUPERCAP.2
